Commit message: panes

File: URDF/tree.urdf (robot description, URDF)
Before this commit: robot None, 100 links, 99 joints
Links:
- removed link link_22
- removed link link_23
- removed link link_24
- removed link link_25
- removed link link_26
- removed link link_27
- removed link link_28
- removed link link_29
- removed link link_30
- removed link link_31
- removed link link_32
- removed link link_33
- removed link link_34
- removed link link_35
- removed link link_36
- removed link link_37
- removed link link_38
- removed link link_39
- removed link link_40
- removed link link_41
- removed link link_42
- removed link link_43
- removed link link_44
- removed link link_45
- removed link link_46
- removed link link_47
- removed link link_48
- removed link link_49
- removed link link_50
- removed link link_51
- removed link link_52
- removed link link_53
- removed link link_54
- removed link link_55
- removed link link_56
- removed link link_57
- removed link link_58
- removed link link_59
- removed link link_60
- removed link link_61
- removed link link_62
- removed link link_63
- removed link link_64
- removed link link_65
- removed link link_66
- removed link link_67
- removed link link_68
- removed link link_69
- removed link link_70
- removed link link_71
- removed link link_72
- removed link link_73
- removed link link_74
- removed link link_75
- removed link link_76
- removed link link_77
- removed link link_78
- removed link link_79
- removed link link_80
- removed link link_81
- removed link link_82
- removed link link_83
- removed link link_84
- removed link link_85
- removed link link_86
- removed link link_87
- removed link link_88
- removed link link_89
- removed link link_90
- removed link link_91
- removed link link_92
- removed link link_93
- removed link link_94
- removed link link_95
- removed link link_96
- removed link link_97
- removed link link_98
- removed link link_99
Joints:
- removed joint joint_22
- removed joint joint_23
- removed joint joint_24
- removed joint joint_25
- removed joint joint_26
- removed joint joint_27
- removed joint joint_28
- removed joint joint_29
- removed joint joint_30
- removed joint joint_31
- removed joint joint_32
- removed joint joint_33
- removed joint joint_34
- removed joint joint_35
- removed joint joint_36
- removed joint joint_37
- removed joint joint_38
- removed joint joint_39
- removed joint joint_40
- removed joint joint_41
- removed joint joint_42
- removed joint joint_43
- removed joint joint_44
- removed joint joint_45
- removed joint joint_46
- removed joint joint_47
- removed joint joint_48
- removed joint joint_49
- removed joint joint_50
- removed joint joint_51
- removed joint joint_52
- removed joint joint_53
- removed joint joint_54
- removed joint joint_55
- removed joint joint_56
- removed joint joint_57
- removed joint joint_58
- removed joint joint_59
- removed joint joint_60
- removed joint joint_61
- removed joint joint_62
- removed joint joint_63
- removed joint joint_64
- removed joint joint_65
- removed joint joint_66
- removed joint joint_67
- removed joint joint_68
- removed joint joint_69
- removed joint joint_70
- removed joint joint_71
- removed joint joint_72
- removed joint joint_73
- removed joint joint_74
- removed joint joint_75
- removed joint joint_76
- removed joint joint_77
- removed joint joint_78
- removed joint joint_79
- removed joint joint_80
- removed joint joint_81
- removed joint joint_82
- removed joint joint_83
- removed joint joint_84
- removed joint joint_85
- removed joint joint_86
- removed joint joint_87
- removed joint joint_88
- removed joint joint_89
- removed joint joint_90
- removed joint joint_91
- removed joint joint_92
- removed joint joint_93
- removed joint joint_94
- removed joint joint_95
- removed joint joint_96
- removed joint joint_97
- removed joint joint_98
- removed joint joint_99
- joint joint_1: origin xyz=0.43729369831377474 0.08994451371454815 0.4245826892881238 rpy=0 0 -1.8079938807913327 -> xyz=-0.015378445409798047 -0.45939835208471147 0.48790687601906657 rpy=0 0 0
- joint joint_10: origin xyz=-0.40504984953377854 -0.39056050197527203 0.6103826131525127 rpy=0 0 -1.3969446384326638 -> xyz=0.20461717272718638 0.26324335251031705 0.44890197398655374 rpy=0 0 0
- joint joint_11: origin xyz=-0.3453225609975549 -0.1082191716766463 0.7202321781127734 rpy=0 0 -1.1361140513292263 -> xyz=-0.3027882446014616 0.3014731856683591 0.3241208560449712 rpy=0 0 0
- joint joint_12: origin xyz=-0.28225237035213746 -0.44385810385139013 0.32645237521687287 rpy=0 0 -0.9119618153160274 -> xyz=0.4829776994029933 0.17452361758269908 0.30661355097753673 rpy=0 0 0
- joint joint_13: origin xyz=-0.17534595942022013 0.15009601256023208 0.4252550256381801 rpy=0 0 1.3406232499643669 -> xyz=0.19654069535732044 0.003935151908275203 0.7160657492479243 rpy=0 0 0
- joint joint_14: origin xyz=0.127519866776445 0.003492532636959922 0.6622519013410946 rpy=0 0 1.5316293634487699 -> xyz=0.4008301434790458 0.3138899731104464 0.3238516635723652 rpy=0 0 0
- joint joint_15: origin xyz=-0.3058660433611595 0.3900527655352094 0.4410535398236083 rpy=0 0 -2.4121012862476965 -> xyz=0.1506607574290587 -0.3223099621317771 0.6409521556977436 rpy=0 0 0
- joint joint_16: origin xyz=-0.09014687682364075 -0.0029718604648545366 0.659478828166973 rpy=0 0 -1.508873330635258 -> xyz=0.10455447670292295 0.4256599010345211 0.41118507660457554 rpy=0 0 0
- joint joint_17: origin xyz=-0.06073340583935538 0.18861685232275438 0.3450161783428519 rpy=0 0 -1.1070496305294348 -> xyz=-0.45330097659000845 0.06499151081226606 0.36362081122025125 rpy=0 0 0
- joint joint_18: origin xyz=0.38708068934358497 0.32687680893295 0.5625141880725818 rpy=0 0 -1.142978648358637 -> xyz=-0.04708622816662411 0.22766715333885523 0.38286785855265104 rpy=0 0 0
- joint joint_19: origin xyz=0.2581788301843735 0.06833047012452365 0.5298808497491772 rpy=0 0 2.5590121681928113 -> xyz=0.18306311776081252 0.3968453840729721 0.37990325054304247 rpy=0 0 0
- joint joint_2: origin xyz=0.37895724824396126 0.20389459276964228 0.5439953404186325 rpy=0 0 -1.0998775193922299 -> xyz=-0.28567380282987975 0.4214016509849856 0.30523246015996686 rpy=0 0 0
- joint joint_20: origin xyz=0.31202906985029577 0.32426404769409667 0.7406269532407586 rpy=0 0 -3.04598187610581 -> xyz=0.07097498846928363 0.3838977012652065 0.6420172069404098 rpy=0 0 0
- joint joint_21: origin xyz=0.38524965029515257 -0.39046034295568965 0.7362133472780885 rpy=0 0 1.1443880381611602 -> xyz=0.33137959748689916 -0.06353283600845361 0.6677245228559818 rpy=0 0 0
- joint joint_3: origin xyz=0.19576271489146513 -0.017184159709579205 0.45742804525973774 rpy=0 0 1.1283475253405002 -> xyz=-0.16130249541987607 0.22941678968421675 0.4319848708525866 rpy=0 0 0
- joint joint_4: origin xyz=0.3778878442797592 -0.22877745394225268 0.3621089127599366 rpy=0 0 -1.9650560318987211 -> xyz=-0.29822209262428745 -0.049232219363947394 0.709222612961334 rpy=0 0 0
- joint joint_5: origin xyz=0.2899136479677886 0.3727697886714758 0.34434922455693295 rpy=0 0 -1.1495859298084647 -> xyz=0.054378440086267466 -0.30734828079664633 0.3061305512921269 rpy=0 0 0
- joint joint_6: origin xyz=-0.1646641918021916 -0.2683142611981645 0.4995287553955674 rpy=0 0 0.7580187812154686 -> xyz=0.13766147265498963 -0.13360704846730298 0.7130358185847183 rpy=0 0 0
- joint joint_7: origin xyz=-0.3287545695921724 0.3292094605317819 0.5696190102949055 rpy=0 0 -0.699032328564754 -> xyz=0.36441860985365915 0.20622561095683567 0.6427584583050867 rpy=0 0 0
- joint joint_8: origin xyz=-0.26577596357864697 -0.3114558698916434 0.7227788885913042 rpy=0 0 -0.5965326896648544 -> xyz=-0.1951362103272033 -0.060685811881114216 0.3360598707459716 rpy=0 0 0
- joint joint_9: origin xyz=0.09142455501616864 -0.4909426432984103 0.4448800092098881 rpy=0 0 0.3976419446755899 -> xyz=-0.13852474093937328 0.43624551559593305 0.3220721443182039 rpy=0 0 0

Commit message: last save

File: URDF/tree.urdf (robot description, URDF)
Before this commit: robot None, 22 links, 21 joints
Joints:
- joint joint_1: origin xyz=-0.015378445409798047 -0.45939835208471147 0.48790687601906657 rpy=0 0 0 -> xyz=0.30642955877433364 0.2761827288813943 0.3 rpy=0 0 0
- joint joint_10: origin xyz=0.20461717272718638 0.26324335251031705 0.44890197398655374 rpy=0 0 0 -> xyz=-0.9524055169375467 0.11806477001187143 0.66 rpy=0 0 0
- joint joint_11: origin xyz=-0.3027882446014616 0.3014731856683591 0.3241208560449712 rpy=0 0 0 -> xyz=-0.04898310914384396 0.3830231409075968 0.7000000000000001 rpy=0 0 0
- joint joint_12: origin xyz=0.4829776994029933 0.17452361758269908 0.30661355097753673 rpy=0 0 0 -> xyz=0.361492728076813 0.05553451246739871 0.7400000000000001 rpy=0 0 0
- joint joint_13: origin xyz=0.19654069535732044 0.003935151908275203 0.7160657492479243 rpy=0 0 0 -> xyz=0.18853656737663016 -0.0876035876602333 0.7800000000000001 rpy=0 0 0
- joint joint_14: origin xyz=0.4008301434790458 0.3138899731104464 0.3238516635723652 rpy=0 0 0 -> xyz=0.8695018679705606 0.3577474465955284 0.8200000000000002 rpy=0 0 0
- joint joint_15: origin xyz=0.1506607574290587 -0.3223099621317771 0.6409521556977436 rpy=0 0 0 -> xyz=-0.040106373113336424 0.6697594884963649 0.8600000000000002 rpy=0 0 0
- joint joint_16: origin xyz=0.10455447670292295 0.4256599010345211 0.41118507660457554 rpy=0 0 0 -> xyz=0.6861117984389933 0.009702252434626857 0.9000000000000002 rpy=0 0 0
- joint joint_17: origin xyz=-0.45330097659000845 0.06499151081226606 0.36362081122025125 rpy=0 0 0 -> xyz=1.0592621573222187 0.43157030422729303 0.9400000000000003 rpy=0 0 0
- joint joint_18: origin xyz=-0.04708622816662411 0.22766715333885523 0.38286785855265104 rpy=0 0 0 -> xyz=-1.1883492815169086 0.19200903175713158 0.9800000000000003 rpy=0 0 0
- joint joint_19: origin xyz=0.18306311776081252 0.3968453840729721 0.37990325054304247 rpy=0 0 0 -> xyz=-1.5535338156854432 0.7489387160267702 1.0200000000000002 rpy=0 0 0
- joint joint_2: origin xyz=-0.28567380282987975 0.4214016509849856 0.30523246015996686 rpy=0 0 0 -> xyz=0.251254117542212 0.0026171477875290006 0.33999999999999997 rpy=0 0 0
- joint joint_20: origin xyz=0.07097498846928363 0.3838977012652065 0.6420172069404098 rpy=0 0 0 -> xyz=-1.3077885698699332 0.6739873456169194 1.0600000000000003 rpy=0 0 0
- joint joint_21: origin xyz=0.33137959748689916 -0.06353283600845361 0.6677245228559818 rpy=0 0 0 -> xyz=0.23068594891447392 0.8650353013152955 1.1000000000000003 rpy=0 0 0
- joint joint_3: origin xyz=-0.16130249541987607 0.22941678968421675 0.4319848708525866 rpy=0 0 0 -> xyz=0.35862421176213877 0.2760954369000074 0.37999999999999995 rpy=0 0 0
- joint joint_4: origin xyz=-0.29822209262428745 -0.049232219363947394 0.709222612961334 rpy=0 0 0 -> xyz=0.20421248735396869 -0.23954136211892318 0.41999999999999993 rpy=0 0 0
- joint joint_5: origin xyz=0.054378440086267466 -0.30734828079664633 0.3061305512921269 rpy=0 0 0 -> xyz=-0.11911701883846515 0.21167361387913075 0.4599999999999999 rpy=0 0 0
- joint joint_6: origin xyz=0.13766147265498963 -0.13360704846730298 0.7130358185847183 rpy=0 0 0 -> xyz=0.1901654642010795 0.36752986938602383 0.4999999999999999 rpy=0 0 0
- joint joint_7: origin xyz=0.36441860985365915 0.20622561095683567 0.6427584583050867 rpy=0 0 0 -> xyz=0.25487682222191976 0.030025892722585545 0.5399999999999999 rpy=0 0 0
- joint joint_8: origin xyz=-0.1951362103272033 -0.060685811881114216 0.3360598707459716 rpy=0 0 0 -> xyz=0.1550404795283724 0.08501459421497715 0.58 rpy=0 0 0
- joint joint_9: origin xyz=-0.13852474093937328 0.43624551559593305 0.3220721443182039 rpy=0 0 0 -> xyz=-0.31634456353033913 0.13182877903390589 0.62 rpy=0 0 0

Commit message: update

File: URDF/tree.urdf (robot description, URDF)
Before this commit: robot None, 22 links, 21 joints
Links:
- removed link link_15
- removed link link_16
- removed link link_17
- removed link link_18
- removed link link_19
- removed link link_20
- removed link link_21
Joints:
- removed joint joint_15
- removed joint joint_16
- removed joint joint_17
- removed joint joint_18
- removed joint joint_19
- removed joint joint_20
- removed joint joint_21
- joint joint_1: origin xyz=0.30642955877433364 0.2761827288813943 0.3 rpy=0 0 0 -> xyz=0.2971076566791907 0.019375247902030962 0.3 rpy=0 0 0
- joint joint_10: origin xyz=-0.9524055169375467 0.11806477001187143 0.66 rpy=0 0 0 -> xyz=0.598486907372207 0.2204388830255991 0.66 rpy=0 0 0
- joint joint_11: origin xyz=-0.04898310914384396 0.3830231409075968 0.7000000000000001 rpy=0 0 0 -> xyz=0.7523874610157555 -0.3353426061708675 0.7000000000000001 rpy=0 0 0
- joint joint_12: origin xyz=0.361492728076813 0.05553451246739871 0.7400000000000001 rpy=0 0 0 -> xyz=1.0112308494454993 -0.17276449387842258 0.7400000000000001 rpy=0 0 0
- joint joint_13: origin xyz=0.18853656737663016 -0.0876035876602333 0.7800000000000001 rpy=0 0 0 -> xyz=-0.2806595307245906 -0.2681638375596923 0.7800000000000001 rpy=0 0 0
- joint joint_14: origin xyz=0.8695018679705606 0.3577474465955284 0.8200000000000002 rpy=0 0 0 -> xyz=-0.035030175582710266 0.4451379147582656 0.8200000000000002 rpy=0 0 0
- joint joint_2: origin xyz=0.251254117542212 0.0026171477875290006 0.33999999999999997 rpy=0 0 0 -> xyz=-0.441983812745443 0.08856549096131108 0.33999999999999997 rpy=0 0 0
- joint joint_3: origin xyz=0.35862421176213877 0.2760954369000074 0.37999999999999995 rpy=0 0 0 -> xyz=0.2266337074523982 0.218802190114796 0.37999999999999995 rpy=0 0 0
- joint joint_4: origin xyz=0.20421248735396869 -0.23954136211892318 0.41999999999999993 rpy=0 0 0 -> xyz=-0.2055237946273366 -0.23417557040509318 0.41999999999999993 rpy=0 0 0
- joint joint_5: origin xyz=-0.11911701883846515 0.21167361387913075 0.4599999999999999 rpy=0 0 0 -> xyz=-0.5926359773403709 0.2740060390417969 0.4599999999999999 rpy=0 0 0
- joint joint_6: origin xyz=0.1901654642010795 0.36752986938602383 0.4999999999999999 rpy=0 0 0 -> xyz=0.08621906137477997 -0.04080739567094682 0.4999999999999999 rpy=0 0 0
- joint joint_7: origin xyz=0.25487682222191976 0.030025892722585545 0.5399999999999999 rpy=0 0 0 -> xyz=-0.7737419403019059 -0.2514926582356516 0.5399999999999999 rpy=0 0 0
- joint joint_8: origin xyz=0.1550404795283724 0.08501459421497715 0.58 rpy=0 0 0 -> xyz=0.2223375333881843 -0.26747690380654165 0.58 rpy=0 0 0
- joint joint_9: origin xyz=-0.31634456353033913 0.13182877903390589 0.62 rpy=0 0 0 -> xyz=0.6884548399916925 0.15411570712390787 0.62 rpy=0 0 0
